Commit message: Fixes for gripper URDF.

File: urdf/a750_rev1.urdf (robot description, URDF)
Before this commit: robot a750-rev1, 8 links, 7 joints
Links:
- removed link link7
- added link gripper_base
- added link left_finger_link; collision mesh filename=package://a750_description/meshes/a750_rev1/collision_finge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 scale=0.001 0.001 0.001; visual mesh filename=package://a750_description/meshes/a750_rev1/finger.stl scale=0.001 0.001 0.001
- added link right_finger_link; collision mesh filename=package://a750_description/meshes/a750_rev1/collision_finge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 scale=0.001 0.001 0.001; visual mesh filename=package://a750_description/meshes/a750_rev1/finger.stl scale=0.001 0.001 0.001
- link link6: geometry collision mesh filename=package://a750_description/meshes/a750_rev1/collision_link6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 scale=0.001 0.001 0.001; visual mesh filename=package://a750_description/meshes/a750_rev1/link6.stl scale=0.001 0.001 0.001
Joints:
- removed joint gripper
- added joint finger: type prismatic, parent gripper_base, child left_finger_link, origin xyz=0.0 0.0 0.0 rpy=0.0 -0.0 0.0, axis 1. 0. 0., limit lower=0.02 upper=0.06 effort=100.0 velocity=255.0
- added joint finger_mimic: type prismatic, parent gripper_base, child right_finger_link, origin xyz=0.0 0.0 0.0 rpy=0.0 -0.0 0.0, axis 1. 0. 0., limit lower=0.02 upper=0.06 effort=100.0 velocity=255.0, mimic joint=finger multiplier=-1.0 offset=0.0
- added joint wrist_to_gripper: type fixed, parent link6, child gripper_base, origin xyz=0.076 0.0 0.0 rpy=-1.5707963267948966 -0.0 -1.5707963267948966, axis 1. 0. 0.

Commit message: update

File: urdf/a750_rev1.urdf (robot description, URDF)
Before this commit: robot a750-rev1, 10 links, 9 joints
Links:
- link left_finger_link: mass None -> 0.04432657029800724
- link link1: mass 0.8698633158614087 -> 0.8585205200761918
- link link2: mass 0.8600472375053468 -> 0.855634866219948
- link link3: mass 0.5997741315905328 -> 0.5577548514954243
- link link4: mass 0.5120280784974558 -> 0.5053526719021317
- link link5: mass 0.4322695513477669 -> 0.42503045095273195
- link link6: mass 0.34348005499634865 -> 0.4767489831533607
- link right_finger_link: mass None -> 0.04432657029800724
Joints:
- joint finger: limit lower=0.02 upper=0.06 effort=100.0 velocity=255.0 -> lower=0.018 upper=0.06 effort=100.0 velocity=255.0
- joint finger_mimic: limit lower=0.02 upper=0.06 effort=100.0 velocity=255.0 -> lower=0.018 upper=0.06 effort=100.0 velocity=255.0
- joint joint4: origin xyz=0.0043 0.0 0.20600000000000002 rpy=1.5707963267948966 -1.5707963267948966 0.0 -> xyz=0.0043 0.0 0.166 rpy=1.5707963267948966 -1.5707963267948966 0.0
- joint joint5: origin xyz=0.08750000000000001 0.020800000000000003 0.0 rpy=1.5707963267948966 -0.0 1.5707963267948966 -> xyz=0.1275 0.020800000000000003 0.0 rpy=1.5707963267948966 -0.0 1.5707963267948966
- joint wrist_to_gripper: origin xyz=0.076 0.0 0.0 rpy=-1.5707963267948966 -0.0 -1.5707963267948966 -> xyz=0.076 0.0 0.0 rpy=1.5707963267948966 -0.0 1.5707963267948966
